Commit message: Fixed Rviz open fault

File: urdf/orion5.urdf (robot description, URDF)
Before this commit: robot orion5, 8 links, 7 joints
Links:
- link base_link: geometry visual mesh filename=package://ros_orion5/urdf/stl/base_link_SCALED.stl
- link bicep: geometry visual mesh filename=package://ros_orion5/urdf/stl/bicep_SCALED.stl
- link forearm: geometry visual mesh filename=package://ros_orion5/urdf/stl/forearm_SCALED.stl
- link gripper1: geometry visual mesh filename=package://ros_orion5/urdf/stl/gripper1_SCALED.stl
- link gripper2: geometry visual mesh filename=package://ros_orion5/urdf/stl/gripper2_SCALED.stl
- link hand: geometry visual mesh filename=package://ros_orion5/urdf/stl/hand_SCALED.stl
- link turret: geometry visual mesh filename=package://ros_orion5/urdf/stl/turret_scaled_translated.stl
